File: hardware/rpi-hat/rpi-hat.kicad_pcb (KiCad board)
At the start: 2 copper layers, 65 x 56 mm, 5 parts, among them P1 Conn_02x20_Odd_Even

Commit message: Begin layout
Parts:
- removed MK1, MK2, MK3, MK4: M2.5, MountingHole:MountingHole_2.7mm_M2.5
- removed P1: Conn_02x20_Odd_Even, Connector_PinSocket_2.54mm:PinSocket_2x20_P2.54mm_Vertical
- added ?: M2.5, MountingHole:MountingHole_2.7mm_M2.5, F.Cu at (203.5, 146.4)
- added ?: M2.5, MountingHole:MountingHole_2.7mm_M2.5, F.Cu at (261.5, 146.5)
- added ?: M2.5, MountingHole:MountingHole_2.7mm_M2.5, F.Cu at (203.5, 97.5)
- added ?: M2.5, MountingHole:MountingHole_2.7mm_M2.5, F.Cu at (261.5, 97.5)
- added C1: 220uF, Resistor_SMD:R_0805_2012Metric_Pad1.15x1.40mm_HandSolder, F.Cu at (245.3, 139.3)
- added C2: 47uF, Resistor_SMD:R_1206_3216Metric_Pad1.42x1.75mm_HandSolder, F.Cu at (214.5, 138.7)
- added D1: , zephyrus-iaq:SMBJ5.0A, F.Cu at (211.0, 138.7)
- added F1: MF-MSMF250/X, Fuse:Fuse_1812_4532Metric, F.Cu at (206.9, 138.6)
- added J1: Conn_02x20_Odd_Even__Rpi, Connector_PinHeader_2.54mm:PinHeader_2x20_P2.54mm_Vertical, F.Cu at (208.4, 98.8)
- added J10: Conn_01x02_Male, Connector_PinSocket_2.54mm:PinSocket_1x02_P2.54mm_Vertical, F.Cu at (213.8, 112.3)
- added J2: , SM04B-SRSS-TB_LF__SN_:JST_SM04B-SRSS-TB(LF)(SN), F.Cu at (220.8, 144.7)
- added J3: , SM04B-SRSS-TB_LF__SN_:JST_SM04B-SRSS-TB(LF)(SN), F.Cu at (229.5, 144.7)
- added J4: , SM04B-SRSS-TB_LF__SN_:JST_SM04B-SRSS-TB(LF)(SN), F.Cu at (238.6, 144.9)
- added J5: , S6B-ZR-SM4A-TF_LF__SN_:JST_S6B-ZR-SM4A-TF(LF)(SN), F.Cu at (250.0, 143.9)
- added J6: , S6B-ZR-SM4A-TF_LF__SN_:JST_S6B-ZR-SM4A-TF(LF)(SN), F.Cu at (258.7, 107.6)
- added J7: , S6B-ZR-SM4A-TF_LF__SN_:JST_S6B-ZR-SM4A-TF(LF)(SN), F.Cu at (258.7, 121.8)
- added J8: , S6B-ZR-SM4A-TF_LF__SN_:JST_S6B-ZR-SM4A-TF(LF)(SN), F.Cu at (258.7, 136.0)
- added J9: , 10103594-0001LF:FCI_10103594-0001LF, F.Cu at (211.1, 147.7)
- added R1: 150, Resistor_SMD:R_0805_2012Metric_Pad1.15x1.40mm_HandSolder, F.Cu at (245.3, 137.2)
- added R2: 3.9k, Resistor_SMD:R_0805_2012Metric_Pad1.15x1.40mm_HandSolder, F.Cu at (217.8, 108.8)
- added R3: 3.9k, Resistor_SMD:R_0805_2012Metric_Pad1.15x1.40mm_HandSolder, F.Cu at (217.8, 110.8)
- added R4: 1700, Resistor_SMD:R_0805_2012Metric_Pad1.15x1.40mm_HandSolder, F.Cu at (246.4, 121.6)
- added R5: 10k, Resistor_SMD:R_0805_2012Metric_Pad1.15x1.40mm_HandSolder, F.Cu at (217.8, 106.7)
- added R6: 3300, Resistor_SMD:R_0805_2012Metric_Pad1.15x1.40mm_HandSolder, F.Cu at (248.8, 121.6)
- added R7: DNP, Resistor_SMD:R_0805_2012Metric_Pad1.15x1.40mm_HandSolder, F.Cu at (217.8, 104.7)
- added U1: , MCP3008T-I_SL:SOIC127P600X175-16N, F.Cu at (240.1, 122.3)
- added U2: , SN74LV4T125PWR:SOP65P640X120-14N, F.Cu at (231.2, 108.3)
- added U3: , CAT24C32WI-GT3:SOIC127P600X175-8N, F.Cu at (211.2, 107.5)
Routing:
- net GND: track 0.00 -> 9.94 mm, vias 0 -> 5
- net Net-(F1-Pad2): track 0.00 -> 5.37 mm
- net Net-(C1-Pad1): track 0.00 -> 1.63 mm
- net ADC6: track 0.00 -> 1.40 mm
- added copper zone on F.Cu, net +5V
- added copper zone on B.Cu, net GND
Other:
- outline, holes or cut-outs redrawn
- net class Default: clearance 0.2 -> 0.1524; trace_width 0.2 -> 0.1524; via_dia 0.9 -> 0.6858; via_drill 0.6 -> 0.3302
- rule trace_clearance: 0.2 -> 0.1524
- rule via_min_drill: 0.5 -> 0.3302
- rule via_min_size: 0.8 -> 0.6858
- board text removed: "CAMERA"
