File: Hardware/FanControl.sch (KiCad schematic (older format))
At the start: 9 parts, among them J4 Fan 1, J5 Fan 2, U2 Fan Driver

Commit message: Fix fan control.
Parts:
- removed D2, D3: LED, Diode_SMD:D_0805_2012Metric, symbol zephyrus_iaq:LED
- removed J5: Fan 2, SM02B-SRSS-TB(LF)(SN), symbol zephyrus_iaq:SM02B-SRSS-TB(LF)(SN)
- removed R7, R8: 330, Resistor_SMD:R_0805_2012Metric, symbol zephyrus_iaq:R_US
- J4: value Fan 1 -> Fan
Connections:
- net labels removed: FAN_PWM0
- wire segments 25 -> 20
Other:
- note added: "2-Pin Connector for Fan\n(Unidirectional Control)"
- note removed: "Fan 2-Pin Connectors\n(Unidirectional Control)"
- note removed: "Fan LED"
- moved on the sheet: C3, J4
