File: Hardware/AnalogPortControl.sch (KiCad schematic (older format))
At the start: 28 parts, among them J10 A0, J11 A1, J12 A2, J13 A3, J14 A4, J15 A5, U11 Buffer, U12 Buffer, U9 DAC

Commit message: Update footprint for AD8532, traces, and back silkscreen.
Parts:
- U12: footprint zephyrus-iaq:SOP65P490X110-8N -> zephyrus-iaq:AD8532ARMZ-MSOP8
Changed lines of the file:
@@
 F 0 "U12" H 6850 6270 50  0000 C CNN
 F 1 "Buffer" H 6850 6179 50  0000 C CNB
-F 2 "zephyrus-iaq:SOP65P490X110-8N" H 6550 6250 50  0001 L BNN
+F 2 "zephyrus-iaq:AD8532ARMZ-MSOP8" H 6550 6250 50  0001 L BNN
 F 3 "" H 7650 6450 50  0001 L BNN
 F 4 "MSOP-8 Analog Devices" H 6550 6350 50  0001 L BNN "Field4"

Commit message: AD8532ARMZ Footprint change.
Parts:
- U12: footprint zephyrus-iaq:AD8532ARMZ-MSOP8 -> zephyrus-iaq:SOP65P490X110-8N
Changed lines of the file:
@@
 F 0 "U12" H 6850 6270 50  0000 C CNN
 F 1 "Buffer" H 6850 6179 50  0000 C CNB
-F 2 "zephyrus-iaq:AD8532ARMZ-MSOP8" H 6550 6250 50  0001 L BNN
+F 2 "zephyrus-iaq:SOP65P490X110-8N" H 6550 6250 50  0001 L BNN
 F 3 "" H 7650 6450 50  0001 L BNN
 F 4 "MSOP-8 Analog Devices" H 6550 6350 50  0001 L BNN "Field4"
